File: hardware/gamebuino-hack.brd (EAGLE design)
At the start: 86.4 x 36.8 mm, 28 parts, among them U1 328P, Y1 16MHz

Commit message: Corrected sound output (removed cap)
Parts:
- removed C6: 10mF, myParts:0805
Connections:
- removed net N$2: C6.1, LS1.-
- net SOUND: now also LS1.-; no longer C6.2
Routing:
- net SOUND: track 23.0 -> 27.6 mm
- net N$2: track 3.45 -> 0.00 mm
Changed lines of the file:
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@@
 <attribute name="VALUE" x="58.42" y="10.541" size="0.6096" layer="28" font="vector" ratio="20" rot="MR0" align="top-center"/>
-</element>
-<element name="C6" library="myParts" package="0805" value="10mF" x="68.58" y="31.75" smashed="yes" rot="MR0">
-<attribute name="NAME" x="68.58" y="32.639" size="0.6096" layer="26" font="vector" ratio="20" rot="MR0" align="bottom-center"/>
-<attribute name="VALUE" x="68.58" y="30.861" size="0.6096" layer="28" font="vector" ratio="20" rot="MR0" align="top-center"/>
 </element>
 <element name="S1" library="SparkFun-Switches" package="SWITCH_SPDT_PTH_11.6X4.0MM" value="" x="69.85" y="5.08" smashed="yes" rot="R90">
@@
 <signal name="SOUND">
 <contactref element="U1" pad="5"/>
-<wire x1="67.31" y1="33.274" x2="52.07" y2="33.274" width="0.4064" layer="16"/>
 <wire x1="49.53" y1="30.734" x2="52.07" y2="33.274" width="0.4064" layer="16"/>
 <wire x1="49.53" y1="28.194" x2="49.53" y2="30.734" width="0.4064" layer="16"/>
-<contactref element="C6" pad="2"/>
-<wire x1="67.68" y1="31.75" x2="67.31" y2="32.12" width="0.4064" layer="16"/>
-<wire x1="67.31" y1="32.12" x2="67.31" y2="33.274" width="0.4064" layer="16"/>
+<contactref element="LS1" pad="-"/>
+<wire x1="71.68" y1="29.55" x2="71.68" y2="29.21" width="0.4064" layer="16"/>
+<wire x1="67.956" y1="33.274" x2="71.68" y2="29.55" width="0.4064" layer="16"/>
+<wire x1="52.07" y1="33.274" x2="67.956" y2="33.274" width="0.4064" layer="16"/>
 </signal>
 <signal name="SCK">
@@
 <wire x1="54.61" y1="15.24" x2="54.61" y2="20.574" width="0.4064" layer="16"/>
 </signal>
-<signal name="N$2">
-<contactref element="LS1" pad="-"/>
-<contactref element="C6" pad="1"/>
-<wire x1="69.48" y1="31.75" x2="71.68" y2="29.55" width="0.4064" layer="16"/>
-<wire x1="71.68" y1="29.55" x2="71.68" y2="29.21" width="0.4064" layer="16"/>
-</signal>
 <signal name="V_BATT">
